File: Archive/MAXTempRTDv0.4/MAXTempRTD.sch (KiCad schematic (older format))
At the start: 19 parts, among them J1 J, J2 J, J3 J, J4 J, P1 RTD1, P2 RTD2, P3 OUTPUT, P4 INPUT, U1 MAX31865, U2 MAX31865

Commit message: Updated v1.1 source files
Parts:
- added C1: 0.1u, ~, symbol C_Small
- C2, C3, C4, C5, C6, C7: footprint complib:C_0603 -> ~
- L1: footprint complib:R_0805 -> ~
- P1, P2: footprint complib:SCREW_TERMINAL_4x1 -> ~
- P3: footprint complib:MAX_TEMP_DB -> ~; symbol CONN_02X05 -> CONN_5X2
- P4: footprint complib:MAX_TEMP_DB_inv -> ~; symbol CONN_02X05 -> CONN_5X2
- R1, R2: footprint complib:R_0603 -> ~
- SJ1: renamed from J1; value J -> SJ; footprint complib:JUMPER -> ~; symbol Jumper_NC_Small -> SJ
- SJ2: renamed from J2; value J -> SJ; footprint complib:JUMPER -> ~; symbol Jumper_NC_Small -> SJ
- SJ3: renamed from J3; value J -> SJ; footprint complib:JUMPER -> ~; symbol Jumper_NC_Small -> SJ
- SJ4: renamed from J4; value J -> SJ; footprint complib:JUMPER -> ~; symbol Jumper_NC_Small -> SJ
- U1, U2: footprint complib:QFN20_5x5 -> (none)
Connections:
- wire segments 166 -> 162
Other:
- moved on the sheet: R1, R2
