File: MAXTempTC/MAXTempTC.sch (KiCad schematic (older format))
At the start: 10 parts, among them J1 ThermC1, J2 ThermC2, P5 OUTPUT, P6 INPUT, U3 MAX31855, U4 MAX31855

Commit message: Updated v1.1 source files
Parts:
- removed C11: 0.1u, ~, symbol Csmall
- removed C12: 0.01u, ~, symbol Csmall
- removed U3, U4: MAX31855, symbol MAX31855
- added C10, C2, C7, C8: 0.1u, complib:C_0603, symbol Csmall
- added C3, C4, C5, C6: 0.01u, complib:C_0603, symbol Csmall
- added D1, D2: FAULT, complib:D_0603, symbol LED
- added L1: 100 µH, complib:R_0805, symbol INDUCTOR_SMALL
- added R1, R2, R3, R4, R5, R6: 100R, complib:R_0603, symbol R
- added R7, R8: 330R, complib:R_0603, symbol R
- added U1, U2: MAX31856, complib:TSSOP-14, symbol MAX31856
- C1: renamed from C10; value 0.01u -> 0.1u; footprint ~ -> complib:C_0603
- C9: footprint ~ -> complib:C_0603
- J1, J2: footprint ~ -> complib:PIN_ARRAY_2X1
- P5: footprint ~ -> complib:MAX_TEMP_DB
- P6: footprint ~ -> complib:MAX_TEMP_DB_inv
Connections:
- net 3.3V: now also C9.2, C10.2, L1.2, R7.2, R8.2, U1.8 (DVDD), U2.8 (DVDD); no longer C9.1
- net CS_1: now also U1.9 (~CS)
- net CS_2: now also U2.9 (~CS)
- net GND: now also C9.1, C10.1, C3.1, C4.1, C5.1, C6.1, C7.2, C8.2, U1.1 (AGND), U1.14 (DGND), U2.1 (AGND), U2.14 (DGND); no longer C9.2
- net MISO: now also U1.11 (SDO), U2.11 (SDO)
- net MOSI: now also U1.12 (SDI), U2.12 (SDI)
- net SCLK: now also U1.10 (SCK), U2.10 (SCK)
- net TC+_A: now also R3.1; no longer C1.1
- net TC+_B: now also R4.1
- net TC-_A: now also R1.1, R5.1; no longer C1.2
- net TC-_B: now also R2.1, R6.1
- new net: C1.1, C3.2, R3.2, U1.4 (T-)
- new net: C1.2, C4.2, R1.2, U1.3 (T-)
- new net: D1.2 (K), U1.13 (~FAULT)
- new net: R5.2, U1.2 (BIAS)
- new net: C2.1, C5.2, R4.2, U2.4 (T-)
- new net: C2.2, C6.2, R2.2, U2.3 (T-)
- new net: D2.2 (K), U2.13 (~FAULT)
- new net: R6.2, U2.2 (BIAS)
- new net: D1.1 (A), R7.1
- new net: D2.1 (A), R8.1
- new net AVDD: C7.1, C8.1, L1.1, U1.5 (AVDD), U2.5 (AVDD)
- no-connect marks 6 -> 8
Other:
- moved on the sheet: C1, J1, J2, P5, P6
